File: elec/keyboard_steamdeck.kicad_sch (KiCad schematic)
At the start: 112 parts, among them IC1 STM32L052K8U6TR, J2 STLINKV2, J3 USB_C_Receptacle_USB2.0, U2 AP63203WU

Commit message: corrections
Parts:
- B1, B10, B11, B12, B13, B14, B15, B16, B17, B18, B19, B2, B20, B21, B22, B23, B24, B25, B26, B27, B28, B29, B3, B30, B31, B32, B33, B34, B35, B36, B37, B38, B39, B4, B40, B41, B42, B43, B44, B5, B6, B7, B8, B9: value MX_SW_solder -> MX_SW_solder - DNI
- IC1: Height 0.6 -> (none); Manufacturer (none) -> StMicroelectronic; Manufacturer_Name STMicroelectronics -> (none); Manufacturer_Part_Number STM32L052K8U6TR -> (none); Mouser Part Number 511-STM32L052K8U6TR -> (none); Mouser Price/Stock https://www.mouser.co.uk/ProductDetail/STMicroelectronics/S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 -> (none); SKU (none) -> 497-18814-1-ND; Vendor (none) -> Digikey
- J2: value STLINKV2 -> STLINKV2 - DNI
- J3: Manufacturer (none) -> Molex; SKU (none) -> 900-2130830005CT-ND; Vendor (none) -> Digikey
Connections:
- net C1: now also IC1.20 (PA10); no longer IC1.3 (PC15-OSC32_OUT)
- net C10: now also IC1.8 (PA2); no longer IC1.25 (PA15)
- net C11: now also IC1.28 (PB5); no longer IC1.8 (PA2)
- net C2: now also IC1.19 (PA9); no longer IC1.7 (PA1)
- net C3: now also IC1.18 (PA8); no longer IC1.32 (PB8)
- net C4: now also IC1.14 (PB0); no longer IC1.6 (PA0)
- net C5: now also IC1.13 (PA7); no longer IC1.30 (PB7)
- net C6: now also IC1.12 (PA6); no longer IC1.29 (PB6)
- net C7: now also IC1.11 (PA5); no longer IC1.28 (PB5)
- net C8: now also IC1.10 (PA4); no longer IC1.27 (PB4)
- net C9: now also IC1.9 (PA3); no longer IC1.26 (PB3)
- net D+: now also D46.3 (K2); no longer D46.4 (K3)
- net D-: now also D46.1 (K1); no longer D46.3 (K2)
- net L1: now also IC1.16 (PB2); no longer IC1.2 (PC14-OSC32_IN)
- net L2: now also IC1.15 (PB1); no longer IC1.20 (PA10)
- net L3: now also IC1.30 (PB7); no longer IC1.19 (PA9)
- net L4: now also IC1.29 (PB6); no longer IC1.18 (PA8)
- no-connect marks 3 -> 11

Commit message: Finish
Parts:
- B1: Item (none) -> 1; MPN (none) -> MX2A-L1NN; Manufacturer (none) -> cherrymx; SKU (none) -> 39810772959301; Type (none) -> thru-hole; URL (none) -> https://boutique-keycaps.com/products/cherry-mx-red?variant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; Vendor (none) -> boutique-keycaps
- B10: Item (none) -> 10; MPN (none) -> MX2A-L1NN; Manufacturer (none) -> cherrymx; SKU (none) -> 39810772959301; Type (none) -> thru-hole; URL (none) -> https://boutique-keycaps.com/products/cherry-mx-red?variant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; Vendor (none) -> boutique-keycaps
- B11: Item (none) -> 11; MPN (none) -> MX2A-L1NN; Manufacturer (none) -> cherrymx; SKU (none) -> 39810772959301; Type (none) -> thru-hole; URL (none) -> https://boutique-keycaps.com/products/cherry-mx-red?variant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; Vendor (none) -> boutique-keycaps
- B12: Item (none) -> 12; MPN (none) -> MX2A-L1NN; Manufacturer (none) -> cherrymx; SKU (none) -> 39810772959301; Type (none) -> thru-hole; URL (none) -> https://boutique-keycaps.com/products/cherry-mx-red?variant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; Vendor (none) -> boutique-keycaps
- B13: Item (none) -> 13; MPN (none) -> MX2A-L1NN; Manufacturer (none) -> cherrymx; SKU (none) -> 39810772959301; Type (none) -> thru-hole; URL (none) -> https://boutique-keycaps.com/products/cherry-mx-red?variant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; Vendor (none) -> boutique-keycaps
- B14: Item (none) -> 14; MPN (none) -> MX2A-L1NN; Manufacturer (none) -> cherrymx; SKU (none) -> 39810772959301; Type (none) -> thru-hole; URL (none) -> https://boutique-keycaps.com/products/cherry-mx-red?variant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; Vendor (none) -> boutique-keycaps
- B15: Item (none) -> 15; MPN (none) -> MX2A-L1NN; Manufacturer (none) -> cherrymx; SKU (none) -> 39810772959301; Type (none) -> thru-hole; URL (none) -> https://boutique-keycaps.com/products/cherry-mx-red?variant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; Vendor (none) -> boutique-keycaps
- B16: Item (none) -> 16; MPN (none) -> MX2A-L1NN; Manufacturer (none) -> cherrymx; SKU (none) -> 39810772959301; Type (none) -> thru-hole; URL (none) -> https://boutique-keycaps.com/products/cherry-mx-red?variant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; Vendor (none) -> boutique-keycaps
- B17: Item (none) -> 17; MPN (none) -> MX2A-L1NN; Manufacturer (none) -> cherrymx; SKU (none) -> 39810772959301; Type (none) -> thru-hole; URL (none) -> https://boutique-keycaps.com/products/cherry-mx-red?variant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; Vendor (none) -> boutique-keycaps
- B18: Item (none) -> 18; MPN (none) -> MX2A-L1NN; Manufacturer (none) -> cherrymx; SKU (none) -> 39810772959301; Type (none) -> thru-hole; URL (none) -> https://boutique-keycaps.com/products/cherry-mx-red?variant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; Vendor (none) -> boutique-keycaps
- B19: Item (none) -> 19; MPN (none) -> MX2A-L1NN; Manufacturer (none) -> cherrymx; SKU (none) -> 39810772959301; Type (none) -> thru-hole; URL (none) -> https://boutique-keycaps.com/products/cherry-mx-red?variant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; Vendor (none) -> boutique-keycaps
- B2: Item (none) -> 2; MPN (none) -> MX2A-L1NN; Manufacturer (none) -> cherrymx; SKU (none) -> 39810772959301; Type (none) -> thru-hole; URL (none) -> https://boutique-keycaps.com/products/cherry-mx-red?variant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; Vendor (none) -> boutique-keycaps
- B20: Item (none) -> 20; MPN (none) -> MX2A-L1NN; Manufacturer (none) -> cherrymx; SKU (none) -> 39810772959301; Type (none) -> thru-hole; URL (none) -> https://boutique-keycaps.com/products/cherry-mx-red?variant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; Vendor (none) -> boutique-keycaps
- B21: Item (none) -> 21; MPN (none) -> MX2A-L1NN; Manufacturer (none) -> cherrymx; SKU (none) -> 39810772959301; Type (none) -> thru-hole; URL (none) -> https://boutique-keycaps.com/products/cherry-mx-red?variant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; Vendor (none) -> boutique-keycaps
- B22: Item (none) -> 22; MPN (none) -> MX2A-L1NN; Manufacturer (none) -> cherrymx; SKU (none) -> 39810772959301; Type (none) -> thru-hole; URL (none) -> https://boutique-keycaps.com/products/cherry-mx-red?variant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; Vendor (none) -> boutique-keycaps
- B23: Item (none) -> 23; MPN (none) -> MX2A-L1NN; Manufacturer (none) -> cherrymx; SKU (none) -> 39810772959301; Type (none) -> thru-hole; URL (none) -> https://boutique-keycaps.com/products/cherry-mx-red?variant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; Vendor (none) -> boutique-keycaps
- B24: Item (none) -> 24; MPN (none) -> MX2A-L1NN; Manufacturer (none) -> cherrymx; SKU (none) -> 39810772959301; Type (none) -> thru-hole; URL (none) -> https://boutique-keycaps.com/products/cherry-mx-red?variant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; Vendor (none) -> boutique-keycaps
- B25: Item (none) -> 25; MPN (none) -> MX2A-L1NN; Manufacturer (none) -> cherrymx; SKU (none) -> 39810772959301; Type (none) -> thru-hole; URL (none) -> https://boutique-keycaps.com/products/cherry-mx-red?variant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; Vendor (none) -> boutique-keycaps
- B26: Item (none) -> 26; MPN (none) -> MX2A-L1NN; Manufacturer (none) -> cherrymx; SKU (none) -> 39810772959301; Type (none) -> thru-hole; URL (none) -> https://boutique-keycaps.com/products/cherry-mx-red?variant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; Vendor (none) -> boutique-keycaps
- B27: Item (none) -> 27; MPN (none) -> MX2A-L1NN; Manufacturer (none) -> cherrymx; SKU (none) -> 39810772959301; Type (none) -> thru-hole; URL (none) -> https://boutique-keycaps.com/products/cherry-mx-red?variant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; Vendor (none) -> boutique-keycaps
- B28: Item (none) -> 28; MPN (none) -> MX2A-L1NN; Manufacturer (none) -> cherrymx; SKU (none) -> 39810772959301; Type (none) -> thru-hole; URL (none) -> https://boutique-keycaps.com/products/cherry-mx-red?variant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; Vendor (none) -> boutique-keycaps
- B29: Item (none) -> 29; MPN (none) -> MX2A-L1NN; Manufacturer (none) -> cherrymx; SKU (none) -> 39810772959301; Type (none) -> thru-hole; URL (none) -> https://boutique-keycaps.com/products/cherry-mx-red?variant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; Vendor (none) -> boutique-keycaps
- B3: Item (none) -> 3; MPN (none) -> MX2A-L1NN; Manufacturer (none) -> cherrymx; SKU (none) -> 39810772959301; Type (none) -> thru-hole; URL (none) -> https://boutique-keycaps.com/products/cherry-mx-red?variant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; Vendor (none) -> boutique-keycaps
- B30: Item (none) -> 30; MPN (none) -> MX2A-L1NN; Manufacturer (none) -> cherrymx; SKU (none) -> 39810772959301; Type (none) -> thru-hole; URL (none) -> https://boutique-keycaps.com/products/cherry-mx-red?variant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; Vendor (none) -> boutique-keycaps
- B31: Item (none) -> 31; MPN (none) -> MX2A-L1NN; Manufacturer (none) -> cherrymx; SKU (none) -> 39810772959301; Type (none) -> thru-hole; URL (none) -> https://boutique-keycaps.com/products/cherry-mx-red?variant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; Vendor (none) -> boutique-keycaps
- B32: Item (none) -> 32; MPN (none) -> MX2A-L1NN; Manufacturer (none) -> cherrymx; SKU (none) -> 39810772959301; Type (none) -> thru-hole; URL (none) -> https://boutique-keycaps.com/products/cherry-mx-red?variant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; Vendor (none) -> boutique-keycaps
- B33: Item (none) -> 33; MPN (none) -> MX2A-L1NN; Manufacturer (none) -> cherrymx; SKU (none) -> 39810772959301; Type (none) -> thru-hole; URL (none) -> https://boutique-keycaps.com/products/cherry-mx-red?variant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; Vendor (none) -> boutique-keycaps
- B34: Item (none) -> 34; MPN (none) -> MX2A-L1NN; Manufacturer (none) -> cherrymx; SKU (none) -> 39810772959301; Type (none) -> thru-hole; URL (none) -> https://boutique-keycaps.com/products/cherry-mx-red?variant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; Vendor (none) -> boutique-keycaps
- B35: Item (none) -> 35; MPN (none) -> MX2A-L1NN; Manufacturer (none) -> cherrymx; SKU (none) -> 39810772959301; Type (none) -> thru-hole; URL (none) -> https://boutique-keycaps.com/products/cherry-mx-red?variant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; Vendor (none) -> boutique-keycaps
- B36: Item (none) -> 36; MPN (none) -> MX2A-L1NN; Manufacturer (none) -> cherrymx; SKU (none) -> 39810772959301; Type (none) -> thru-hole; URL (none) -> https://boutique-keycaps.com/products/cherry-mx-red?variant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; Vendor (none) -> boutique-keycaps
- B37: Item (none) -> 37; MPN (none) -> MX2A-L1NN; Manufacturer (none) -> cherrymx; SKU (none) -> 39810772959301; Type (none) -> thru-hole; URL (none) -> https://boutique-keycaps.com/products/cherry-mx-red?variant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; Vendor (none) -> boutique-keycaps
- B38: Item (none) -> 38; MPN (none) -> MX2A-L1NN; Manufacturer (none) -> cherrymx; SKU (none) -> 39810772959301; Type (none) -> thru-hole; URL (none) -> https://boutique-keycaps.com/products/cherry-mx-red?variant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; Vendor (none) -> boutique-keycaps
- B39: Item (none) -> 39; MPN (none) -> MX2A-L1NN; Manufacturer (none) -> cherrymx; SKU (none) -> 39810772959301; Type (none) -> thru-hole; URL (none) -> https://boutique-keycaps.com/products/cherry-mx-red?variant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; Vendor (none) -> boutique-keycaps
- B4: Item (none) -> 4; MPN (none) -> MX2A-L1NN; Manufacturer (none) -> cherrymx; SKU (none) -> 39810772959301; Type (none) -> thru-hole; URL (none) -> https://boutique-keycaps.com/products/cherry-mx-red?variant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; Vendor (none) -> boutique-keycaps
- B40: Item (none) -> 40; MPN (none) -> MX2A-L1NN; Manufacturer (none) -> cherrymx; SKU (none) -> 39810772959301; Type (none) -> thru-hole; URL (none) -> https://boutique-keycaps.com/products/cherry-mx-red?variant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; Vendor (none) -> boutique-keycaps
- B41: Item (none) -> 41; MPN (none) -> MX2A-L1NN; Manufacturer (none) -> cherrymx; SKU (none) -> 39810772959301; Type (none) -> thru-hole; URL (none) -> https://boutique-keycaps.com/products/cherry-mx-red?variant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; Vendor (none) -> boutique-keycaps
- B42: Item (none) -> 42; MPN (none) -> MX2A-L1NN; Manufacturer (none) -> cherrymx; SKU (none) -> 39810772959301; Type (none) -> thru-hole; URL (none) -> https://boutique-keycaps.com/products/cherry-mx-red?variant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; Vendor (none) -> boutique-keycaps
- B43: Item (none) -> 43; MPN (none) -> MX2A-L1NN; Manufacturer (none) -> cherrymx; SKU (none) -> 39810772959301; Type (none) -> thru-hole; URL (none) -> https://boutique-keycaps.com/products/cherry-mx-red?variant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; Vendor (none) -> boutique-keycaps
- B44: Item (none) -> 44; MPN (none) -> MX2A-L1NN; Manufacturer (none) -> cherrymx; SKU (none) -> 39810772959301; Type (none) -> thru-hole; URL (none) -> https://boutique-keycaps.com/products/cherry-mx-red?variant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; Vendor (none) -> boutique-keycaps
- B5: Item (none) -> 5; MPN (none) -> MX2A-L1NN; Manufacturer (none) -> cherrymx; SKU (none) -> 39810772959301; Type (none) -> thru-hole; URL (none) -> https://boutique-keycaps.com/products/cherry-mx-red?variant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; Vendor (none) -> boutique-keycaps
- B6: Item (none) -> 6; MPN (none) -> MX2A-L1NN; Manufacturer (none) -> cherrymx; SKU (none) -> 39810772959301; Type (none) -> thru-hole; URL (none) -> https://boutique-keycaps.com/products/cherry-mx-red?variant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; Vendor (none) -> boutique-keycaps
- B7: Item (none) -> 7; MPN (none) -> MX2A-L1NN; Manufacturer (none) -> cherrymx; SKU (none) -> 39810772959301; Type (none) -> thru-hole; URL (none) -> https://boutique-keycaps.com/products/cherry-mx-red?variant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; Vendor (none) -> boutique-keycaps
- B8: Item (none) -> 8; MPN (none) -> MX2A-L1NN; Manufacturer (none) -> cherrymx; SKU (none) -> 39810772959301; Type (none) -> thru-hole; URL (none) -> https://boutique-keycaps.com/products/cherry-mx-red?variant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; Vendor (none) -> boutique-keycaps
- B9: Item (none) -> 9; MPN (none) -> MX2A-L1NN; Manufacturer (none) -> cherrymx; SKU (none) -> 39810772959301; Type (none) -> thru-hole; URL (none) -> https://boutique-keycaps.com/products/cherry-mx-red?variant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; Vendor (none) -> boutique-keycaps
- C1: Item (none) -> 45; MPN (none) -> CC0402ZRY5V7BB104; Manufacturer (none) -> YAGEO; Package (none) -> 402; SKU (none) -> 311-1047-1-ND; Type (none) -> SMD; URL (none) -> https://www.digikey.fr/en/products/detail/yageo/CC0402ZRY5V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; Vendor (none) -> Digikey
- C10: Item (none) -> 49; MPN (none) -> CC0402ZRY5V7BB104; Manufacturer (none) -> YAGEO; Package (none) -> 402; SKU (none) -> 311-1047-1-ND; Type (none) -> SMD; URL (none) -> https://www.digikey.fr/en/products/detail/yageo/CC0402ZRY5V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; Vendor (none) -> Digikey
- C2: Item (none) -> 46; MPN (none) -> CC0402ZRY5V7BB104; Manufacturer (none) -> YAGEO; Package (none) -> 402; SKU (none) -> 311-1047-1-ND; Type (none) -> SMD; URL (none) -> https://www.digikey.fr/en/products/detail/yageo/CC0402ZRY5V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; Vendor (none) -> Digikey
- C3: Item (none) -> 47; MPN (none) -> CC0402ZRY5V7BB104; Manufacturer (none) -> YAGEO; Package (none) -> 402; SKU (none) -> 311-1047-1-ND; Type (none) -> SMD; URL (none) -> https://www.digikey.fr/en/products/detail/yageo/CC0402ZRY5V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; Vendor (none) -> Digikey
- C4: Item (none) -> 50; MPN (none) -> GMC21X7R106K16NT; Manufacturer (none) -> Cal-Chip Electronics, Inc.; Package (none) -> 805; SKU (none) -> 4713-GMC21X7R106K16NTCT-ND; Type (none) -> SMD; URL (none) -> https://www.digikey.fr/en/products/detail/cal-chip-electron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; Vendor (none) -> Digikey
- C5: Item (none) -> 51; MPN (none) -> GMC21X7R106K16NT; Manufacturer (none) -> Cal-Chip Electronics, Inc.; Package (none) -> 805; SKU (none) -> 4713-GMC21X7R106K16NTCT-ND; Type (none) -> SMD; URL (none) -> https://www.digikey.fr/en/products/detail/cal-chip-electron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; Vendor (none) -> Digikey
- C6: Item (none) -> 48; MPN (none) -> CC0402ZRY5V7BB104; Manufacturer (none) -> YAGEO; Package (none) -> 402; SKU (none) -> 311-1047-1-ND; Type (none) -> SMD; URL (none) -> https://www.digikey.fr/en/products/detail/yageo/CC0402ZRY5V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; Vendor (none) -> Digikey
- C8: Item (none) -> 52; MPN (none) -> GMC21X7R106K16NT; Manufacturer (none) -> Cal-Chip Electronics, Inc.; Package (none) -> 805; SKU (none) -> 4713-GMC21X7R106K16NTCT-ND; Type (none) -> SMD; URL (none) -> https://www.digikey.fr/en/products/detail/cal-chip-electron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; Vendor (none) -> Digikey
- C9: Item (none) -> 53; MPN (none) -> GMC21X7R106K16NT; Manufacturer (none) -> Cal-Chip Electronics, Inc.; Package (none) -> 805; SKU (none) -> 4713-GMC21X7R106K16NTCT-ND; Type (none) -> SMD; URL (none) -> https://www.digikey.fr/en/products/detail/cal-chip-electron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; Vendor (none) -> Digikey
- D1: Item (none) -> 54; MPN (none) -> 1N4148WX-TP; Manufacturer (none) -> Micro Commercial Co; Package (none) -> SOD-323; SKU (none) -> 1N4148WXTPMSCT-ND; Type (none) -> SMD; URL (none) -> https://www.digikey.fr/en/products/detail/micro-commercial-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; Vendor (none) -> Digikey
- D10: Item (none) -> 63; MPN (none) -> 1N4148WX-TP; Manufacturer (none) -> Micro Commercial Co; Package (none) -> SOD-323; SKU (none) -> 1N4148WXTPMSCT-ND; Type (none) -> SMD; URL (none) -> https://www.digikey.fr/en/products/detail/micro-commercial-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; Vendor (none) -> Digikey
- D11: Item (none) -> 64; MPN (none) -> 1N4148WX-TP; Manufacturer (none) -> Micro Commercial Co; Package (none) -> SOD-323; SKU (none) -> 1N4148WXTPMSCT-ND; Type (none) -> SMD; URL (none) -> https://www.digikey.fr/en/products/detail/micro-commercial-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; Vendor (none) -> Digikey
- D12: Item (none) -> 65; MPN (none) -> 1N4148WX-TP; Manufacturer (none) -> Micro Commercial Co; Package (none) -> SOD-323; SKU (none) -> 1N4148WXTPMSCT-ND; Type (none) -> SMD; URL (none) -> https://www.digikey.fr/en/products/detail/micro-commercial-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; Vendor (none) -> Digikey
- D13: Item (none) -> 66; MPN (none) -> 1N4148WX-TP; Manufacturer (none) -> Micro Commercial Co; Package (none) -> SOD-323; SKU (none) -> 1N4148WXTPMSCT-ND; Type (none) -> SMD; URL (none) -> https://www.digikey.fr/en/products/detail/micro-commercial-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; Vendor (none) -> Digikey
- D14: Item (none) -> 67; MPN (none) -> 1N4148WX-TP; Manufacturer (none) -> Micro Commercial Co; Package (none) -> SOD-323; SKU (none) -> 1N4148WXTPMSCT-ND; Type (none) -> SMD; URL (none) -> https://www.digikey.fr/en/products/detail/micro-commercial-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; Vendor (none) -> Digikey
- D15: Item (none) -> 68; MPN (none) -> 1N4148WX-TP; Manufacturer (none) -> Micro Commercial Co; Package (none) -> SOD-323; SKU (none) -> 1N4148WXTPMSCT-ND; Type (none) -> SMD; URL (none) -> https://www.digikey.fr/en/products/detail/micro-commercial-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; Vendor (none) -> Digikey
- D16: Item (none) -> 69; MPN (none) -> 1N4148WX-TP; Manufacturer (none) -> Micro Commercial Co; Package (none) -> SOD-323; SKU (none) -> 1N4148WXTPMSCT-ND; Type (none) -> SMD; URL (none) -> https://www.digikey.fr/en/products/detail/micro-commercial-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; Vendor (none) -> Digikey
- D17: Item (none) -> 70; MPN (none) -> 1N4148WX-TP; Manufacturer (none) -> Micro Commercial Co; Package (none) -> SOD-323; SKU (none) -> 1N4148WXTPMSCT-ND; Type (none) -> SMD; URL (none) -> https://www.digikey.fr/en/products/detail/micro-commercial-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; Vendor (none) -> Digikey
- D18: Item (none) -> 71; MPN (none) -> 1N4148WX-TP; Manufacturer (none) -> Micro Commercial Co; Package (none) -> SOD-323; SKU (none) -> 1N4148WXTPMSCT-ND; Type (none) -> SMD; URL (none) -> https://www.digikey.fr/en/products/detail/micro-commercial-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; Vendor (none) -> Digikey
- D19: Item (none) -> 72; MPN (none) -> 1N4148WX-TP; Manufacturer (none) -> Micro Commercial Co; Package (none) -> SOD-323; SKU (none) -> 1N4148WXTPMSCT-ND; Type (none) -> SMD; URL (none) -> https://www.digikey.fr/en/products/detail/micro-commercial-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; Vendor (none) -> Digikey
- D2: Item (none) -> 55; MPN (none) -> 1N4148WX-TP; Manufacturer (none) -> Micro Commercial Co; Package (none) -> SOD-323; SKU (none) -> 1N4148WXTPMSCT-ND; Type (none) -> SMD; URL (none) -> https://www.digikey.fr/en/products/detail/micro-commercial-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; Vendor (none) -> Digikey
- D20: Item (none) -> 73; MPN (none) -> 1N4148WX-TP; Manufacturer (none) -> Micro Commercial Co; Package (none) -> SOD-323; SKU (none) -> 1N4148WXTPMSCT-ND; Type (none) -> SMD; URL (none) -> https://www.digikey.fr/en/products/detail/micro-commercial-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; Vendor (none) -> Digikey
- D21: Item (none) -> 74; MPN (none) -> 1N4148WX-TP; Manufacturer (none) -> Micro Commercial Co; Package (none) -> SOD-323; SKU (none) -> 1N4148WXTPMSCT-ND; Type (none) -> SMD; URL (none) -> https://www.digikey.fr/en/products/detail/micro-commercial-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; Vendor (none) -> Digikey
- D22: Item (none) -> 75; MPN (none) -> 1N4148WX-TP; Manufacturer (none) -> Micro Commercial Co; Package (none) -> SOD-323; SKU (none) -> 1N4148WXTPMSCT-ND; Type (none) -> SMD; URL (none) -> https://www.digikey.fr/en/products/detail/micro-commercial-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; Vendor (none) -> Digikey
- D23: Item (none) -> 76; MPN (none) -> 1N4148WX-TP; Manufacturer (none) -> Micro Commercial Co; Package (none) -> SOD-323; SKU (none) -> 1N4148WXTPMSCT-ND; Type (none) -> SMD; URL (none) -> https://www.digikey.fr/en/products/detail/micro-commercial-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; Vendor (none) -> Digikey
- D24: Item (none) -> 77; MPN (none) -> 1N4148WX-TP; Manufacturer (none) -> Micro Commercial Co; Package (none) -> SOD-323; SKU (none) -> 1N4148WXTPMSCT-ND; Type (none) -> SMD; URL (none) -> https://www.digikey.fr/en/products/detail/micro-commercial-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; Vendor (none) -> Digikey
- D25: Item (none) -> 78; MPN (none) -> 1N4148WX-TP; Manufacturer (none) -> Micro Commercial Co; Package (none) -> SOD-323; SKU (none) -> 1N4148WXTPMSCT-ND; Type (none) -> SMD; URL (none) -> https://www.digikey.fr/en/products/detail/micro-commercial-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; Vendor (none) -> Digikey
- D26: Item (none) -> 79; MPN (none) -> 1N4148WX-TP; Manufacturer (none) -> Micro Commercial Co; Package (none) -> SOD-323; SKU (none) -> 1N4148WXTPMSCT-ND; Type (none) -> SMD; URL (none) -> https://www.digikey.fr/en/products/detail/micro-commercial-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; Vendor (none) -> Digikey
- D27: Item (none) -> 80; MPN (none) -> 1N4148WX-TP; Manufacturer (none) -> Micro Commercial Co; Package (none) -> SOD-323; SKU (none) -> 1N4148WXTPMSCT-ND; Type (none) -> SMD; URL (none) -> https://www.digikey.fr/en/products/detail/micro-commercial-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; Vendor (none) -> Digikey
- D28: Item (none) -> 81; MPN (none) -> 1N4148WX-TP; Manufacturer (none) -> Micro Commercial Co; Package (none) -> SOD-323; SKU (none) -> 1N4148WXTPMSCT-ND; Type (none) -> SMD; URL (none) -> https://www.digikey.fr/en/products/detail/micro-commercial-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; Vendor (none) -> Digikey
- D29: Item (none) -> 82; MPN (none) -> 1N4148WX-TP; Manufacturer (none) -> Micro Commercial Co; Package (none) -> SOD-323; SKU (none) -> 1N4148WXTPMSCT-ND; Type (none) -> SMD; URL (none) -> https://www.digikey.fr/en/products/detail/micro-commercial-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; Vendor (none) -> Digikey
- D3: Item (none) -> 56; MPN (none) -> 1N4148WX-TP; Manufacturer (none) -> Micro Commercial Co; Package (none) -> SOD-323; SKU (none) -> 1N4148WXTPMSCT-ND; Type (none) -> SMD; URL (none) -> https://www.digikey.fr/en/products/detail/micro-commercial-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; Vendor (none) -> Digikey
- D30: Item (none) -> 83; MPN (none) -> 1N4148WX-TP; Manufacturer (none) -> Micro Commercial Co; Package (none) -> SOD-323; SKU (none) -> 1N4148WXTPMSCT-ND; Type (none) -> SMD; URL (none) -> https://www.digikey.fr/en/products/detail/micro-commercial-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; Vendor (none) -> Digikey
- D31: Item (none) -> 84; MPN (none) -> 1N4148WX-TP; Manufacturer (none) -> Micro Commercial Co; Package (none) -> SOD-323; SKU (none) -> 1N4148WXTPMSCT-ND; Type (none) -> SMD; URL (none) -> https://www.digikey.fr/en/products/detail/micro-commercial-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; Vendor (none) -> Digikey
- D32: Item (none) -> 85; MPN (none) -> 1N4148WX-TP; Manufacturer (none) -> Micro Commercial Co; Package (none) -> SOD-323; SKU (none) -> 1N4148WXTPMSCT-ND; Type (none) -> SMD; URL (none) -> https://www.digikey.fr/en/products/detail/micro-commercial-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; Vendor (none) -> Digikey
- D33: Item (none) -> 86; MPN (none) -> 1N4148WX-TP; Manufacturer (none) -> Micro Commercial Co; Package (none) -> SOD-323; SKU (none) -> 1N4148WXTPMSCT-ND; Type (none) -> SMD; URL (none) -> https://www.digikey.fr/en/products/detail/micro-commercial-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; Vendor (none) -> Digikey
- D34: Item (none) -> 87; MPN (none) -> 1N4148WX-TP; Manufacturer (none) -> Micro Commercial Co; Package (none) -> SOD-323; SKU (none) -> 1N4148WXTPMSCT-ND; Type (none) -> SMD; URL (none) -> https://www.digikey.fr/en/products/detail/micro-commercial-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; Vendor (none) -> Digikey
- D35: Item (none) -> 88; MPN (none) -> 1N4148WX-TP; Manufacturer (none) -> Micro Commercial Co; Package (none) -> SOD-323; SKU (none) -> 1N4148WXTPMSCT-ND; Type (none) -> SMD; URL (none) -> https://www.digikey.fr/en/products/detail/micro-commercial-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; Vendor (none) -> Digikey
- D36: Item (none) -> 89; MPN (none) -> 1N4148WX-TP; Manufacturer (none) -> Micro Commercial Co; Package (none) -> SOD-323; SKU (none) -> 1N4148WXTPMSCT-ND; Type (none) -> SMD; URL (none) -> https://www.digikey.fr/en/products/detail/micro-commercial-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; Vendor (none) -> Digikey
- D37: Item (none) -> 90; MPN (none) -> 1N4148WX-TP; Manufacturer (none) -> Micro Commercial Co; Package (none) -> SOD-323; SKU (none) -> 1N4148WXTPMSCT-ND; Type (none) -> SMD; URL (none) -> https://www.digikey.fr/en/products/detail/micro-commercial-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; Vendor (none) -> Digikey
- D38: Item (none) -> 91; MPN (none) -> 1N4148WX-TP; Manufacturer (none) -> Micro Commercial Co; Package (none) -> SOD-323; SKU (none) -> 1N4148WXTPMSCT-ND; Type (none) -> SMD; URL (none) -> https://www.digikey.fr/en/products/detail/micro-commercial-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; Vendor (none) -> Digikey
- D39: Item (none) -> 92; MPN (none) -> 1N4148WX-TP; Manufacturer (none) -> Micro Commercial Co; Package (none) -> SOD-323; SKU (none) -> 1N4148WXTPMSCT-ND; Type (none) -> SMD; URL (none) -> https://www.digikey.fr/en/products/detail/micro-commercial-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; Vendor (none) -> Digikey
- D4: Item (none) -> 57; MPN (none) -> 1N4148WX-TP; Manufacturer (none) -> Micro Commercial Co; Package (none) -> SOD-323; SKU (none) -> 1N4148WXTPMSCT-ND; Type (none) -> SMD; URL (none) -> https://www.digikey.fr/en/products/detail/micro-commercial-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; Vendor (none) -> Digikey
- D40: Item (none) -> 93; MPN (none) -> 1N4148WX-TP; Manufacturer (none) -> Micro Commercial Co; Package (none) -> SOD-323; SKU (none) -> 1N4148WXTPMSCT-ND; Type (none) -> SMD; URL (none) -> https://www.digikey.fr/en/products/detail/micro-commercial-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; Vendor (none) -> Digikey
- D41: Item (none) -> 94; MPN (none) -> 1N4148WX-TP; Manufacturer (none) -> Micro Commercial Co; Package (none) -> SOD-323; SKU (none) -> 1N4148WXTPMSCT-ND; Type (none) -> SMD; URL (none) -> https://www.digikey.fr/en/products/detail/micro-commercial-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; Vendor (none) -> Digikey
- D42: Item (none) -> 95; MPN (none) -> 1N4148WX-TP; Manufacturer (none) -> Micro Commercial Co; Package (none) -> SOD-323; SKU (none) -> 1N4148WXTPMSCT-ND; Type (none) -> SMD; URL (none) -> https://www.digikey.fr/en/products/detail/micro-commercial-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; Vendor (none) -> Digikey
- D43: Item (none) -> 96; MPN (none) -> 1N4148WX-TP; Manufacturer (none) -> Micro Commercial Co; Package (none) -> SOD-323; SKU (none) -> 1N4148WXTPMSCT-ND; Type (none) -> SMD; URL (none) -> https://www.digikey.fr/en/products/detail/micro-commercial-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; Vendor (none) -> Digikey
- D44: Item (none) -> 97; MPN (none) -> 1N4148WX-TP; Manufacturer (none) -> Micro Commercial Co; Package (none) -> SOD-323; SKU (none) -> 1N4148WXTPMSCT-ND; Type (none) -> SMD; URL (none) -> https://www.digikey.fr/en/products/detail/micro-commercial-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; Vendor (none) -> Digikey
- D46: Item (none) -> 98; MPN (none) -> RCLAMP0503F.TCT; Manufacturer (none) -> Semtech Corporation; Package (none) -> SOT-353; SKU (none) -> RCLAMP0503F.TCTCT-ND; Type (none) -> SMD; URL (none) -> https://www.digikey.fr/en/products/detail/semtech-corporati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; Vendor (none) -> Digikey
- D5: Item (none) -> 58; MPN (none) -> 1N4148WX-TP; Manufacturer (none) -> Micro Commercial Co; Package (none) -> SOD-323; SKU (none) -> 1N4148WXTPMSCT-ND; Type (none) -> SMD; URL (none) -> https://www.digikey.fr/en/products/detail/micro-commercial-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; Vendor (none) -> Digikey
- D6: Item (none) -> 59; MPN (none) -> 1N4148WX-TP; Manufacturer (none) -> Micro Commercial Co; Package (none) -> SOD-323; SKU (none) -> 1N4148WXTPMSCT-ND; Type (none) -> SMD; URL (none) -> https://www.digikey.fr/en/products/detail/micro-commercial-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; Vendor (none) -> Digikey
- D7: Item (none) -> 60; MPN (none) -> 1N4148WX-TP; Manufacturer (none) -> Micro Commercial Co; Package (none) -> SOD-323; SKU (none) -> 1N4148WXTPMSCT-ND; Type (none) -> SMD; URL (none) -> https://www.digikey.fr/en/products/detail/micro-commercial-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; Vendor (none) -> Digikey
- D8: Item (none) -> 61; MPN (none) -> 1N4148WX-TP; Manufacturer (none) -> Micro Commercial Co; Package (none) -> SOD-323; SKU (none) -> 1N4148WXTPMSCT-ND; Type (none) -> SMD; URL (none) -> https://www.digikey.fr/en/products/detail/micro-commercial-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; Vendor (none) -> Digikey
- D9: Item (none) -> 62; MPN (none) -> 1N4148WX-TP; Manufacturer (none) -> Micro Commercial Co; Package (none) -> SOD-323; SKU (none) -> 1N4148WXTPMSCT-ND; Type (none) -> SMD; URL (none) -> https://www.digikey.fr/en/products/detail/micro-commercial-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; Vendor (none) -> Digikey
- FB1: Item (none) -> 99; MPN (none) -> HZ0402A601R-10; Manufacturer (none) -> Laird-Signal Integrity Products; Package (none) -> 402; SKU (none) -> 240-2364-1-ND; Type (none) -> SMD; URL (none) -> https://www.digikey.fr/en/products/detail/laird-signal-inte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; Vendor (none) -> Digikey
- H1: Item (none) -> 100; Manufacturer (none) -> X; Package (none) -> X; SKU (none) -> X; Type (none) -> thru-hole; URL (none) -> X; Vendor (none) -> X
- H2: Item (none) -> 101; Manufacturer (none) -> X; Package (none) -> X; SKU (none) -> X; Type (none) -> thru-hole; URL (none) -> X; Vendor (none) -> X
- H3: Item (none) -> 102; Manufacturer (none) -> X; Package (none) -> X; SKU (none) -> X; Type (none) -> thru-hole; URL (none) -> X; Vendor (none) -> X
- H4: Item (none) -> 103; Manufacturer (none) -> X; Package (none) -> X; SKU (none) -> X; Type (none) -> thru-hole; URL (none) -> X; Vendor (none) -> X
- IC1: Item (none) -> 104; MPN (none) -> STM32L052K8U6TR; Package (none) -> SMD; Type (none) -> SMD; URL (none) -> https://www.digikey.fr/en/products/detail/stmicroelectronic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
- J2: Item (none) -> 105; MPN (none) -> 61300411121; Manufacturer (none) -> Würth Elektronik; Package (none) -> 2.54; SKU (none) -> 732-5317-ND; Type (none) -> thru-hole; URL (none) -> https://www.digikey.fr/en/products/detail/w%C3%BCrth-elektr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; Vendor (none) -> Digikey
- J3: Item (none) -> 106; Package (none) -> Right Angle; Type (none) -> thru-hole; URL (none) -> https://www.digikey.fr/en/products/detail/molex/2130830005/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
- L2: Item (none) -> 107; Manufacturer (none) -> TDK Corporation; Package (none) -> 805; SKU (none) -> 445-6759-1-ND; Type (none) -> SMD; URL (none) -> https://www.digikey.fr/en/products/detail/tdk-corporation/m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; Vendor (none) -> Digikey
- R1: Item (none) -> 108; MPN (none) -> ERA-2AEB103X; Manufacturer (none) -> Panasonic Electronic Components; Package (none) -> 402; SKU (none) -> P10KDCCT-ND; Type (none) -> SMD; URL (none) -> https://www.digikey.fr/en/products/detail/panasonic-electro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; Vendor (none) -> Digikey
- R2: Item (none) -> 109; MPN (none) -> ERA-2AEB103X; Manufacturer (none) -> Panasonic Electronic Components; Package (none) -> 402; SKU (none) -> P10KDCCT-ND; Type (none) -> SMD; URL (none) -> https://www.digikey.fr/en/products/detail/panasonic-electro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; Vendor (none) -> Digikey
- R3: Item (none) -> 110; MPN (none) -> RN73R1ETTP5101B25; Manufacturer (none) -> KOA Speer Electronics, Inc.; Package (none) -> 402; SKU (none) -> 2019-RN73R1ETTP5101B25CT-ND; Type (none) -> SMD; URL (none) -> https://www.digikey.fr/en/products/detail/koa-speer-electro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; Vendor (none) -> Digikey
- R6: Item (none) -> 111; MPN (none) -> RN73R1ETTP5101B25; Manufacturer (none) -> KOA Speer Electronics, Inc.; Package (none) -> 402; SKU (none) -> 2019-RN73R1ETTP5101B25CT-ND; Type (none) -> SMD; URL (none) -> https://www.digikey.fr/en/products/detail/koa-speer-electro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; Vendor (none) -> Digikey
- U2: Item (none) -> 112; MPN (none) -> AP63203WU-7; Manufacturer (none) -> Diodes Incorporated; Package (none) -> SOT-23-6; SKU (none) -> AP63203WU-7DICT-ND; Type (none) -> SMD; URL (none) -> https://www.digikey.fr/en/products/detail/diodes-incorporat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; Vendor (none) -> digikey
Other:
- note added: "MOUNTING"
- company: (none) -> Vincent Bénet & Vincent Legouis
- title: (none) -> KeyBoard SteamDeck
- moved on the sheet: C1, C10, C2, C3, C4, C5, C6, C8, C9, D46, FB1, H1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
