File: elec/keyboard_steamdeck.kicad_sch (KiCad schematic)
At the start: 112 parts, among them IC1 STM32L052K8U6TR, J2 STLINKV2 - DNI, J3 USB_C_Receptacle_USB2.0, U2 AP63203WU

Commit message: ready to order PCB
Parts:
- B1, B10, B11, B12, B13, B14, B15, B16, B17, B18, B19, B2, B20, B21, B22, B23, B24, B25, B26, B27, B28, B29, B3, B30, B31, B32, B33, B34, B35, B36, B37, B38, B39, B4, B40, B41, B42, B43, B44, B5, B6, B7, B8, B9: Package (none) -> X
- C1, C10, C2, C3, C6: MPN CC0402ZRY5V7BB104 -> CC0402KRX7R8BB104; SKU 311-1047-1-ND -> 311-2077-1-ND; URL https://www.digikey.fr/en/products/detail/yageo/CC0402ZRY5V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 -> https://www.digikey.fr/en/products/detail/yageo/cc0402krx7r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
- C4, C5, C8, C9: MPN GMC21X7R106K16NT -> CAP0805 X7R 10UF 10% 16V
- FB1: MPN HZ0402A601R-10 -> PE-0603PFB121ST; Manufacturer Laird-Signal Integrity Products -> Pulse Electronics; SKU 240-2364-1-ND -> 553-2387-1-ND; URL https://www.digikey.fr/en/products/detail/laird-signal-inte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 -> https://www.digikey.fr/en/products/detail/pulse-electronics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
