File: elec/keyboard_steamdeck.kicad_pcb (KiCad board)
At the start: 4 copper layers, 213.4 x 77.8 mm, 112 parts, among them IC1 STM32L052K8U6TR, J2 STLINKV2, J3 USB_C_Receptacle_USB2.0, U2 AP63203WU

Commit message: corrections
Parts:
- B1, B10, B11, B12, B13, B14, B15, B16, B17, B18, B19, B2, B20, B21, B22, B23, B24, B25, B26, B27, B28, B29, B3, B30, B31, B32, B33, B34, B35, B36, B37, B38, B39, B4, B40, B41, B42, B43, B44, B5, B6, B7, B8, B9: value MX_SW_solder -> MX_SW_solder - DNI
- J2: value STLINKV2 -> STLINKV2 - DNI
- moved R1 14.5 mm to (203.8, 38.5), turned to 180 degrees
- moved C6 13.5 mm to (203.8, 37.2), turned to 0 degrees
- moved C5 10.9 mm to (203.5, 34.5), turned to 0 degrees
- moved C1 8.48 mm to (204.0, 32.8), turned to 0 degrees
- moved FB1 7.01 mm to (206.5, 36.0)
- moved C2 6.65 mm to (207.0, 32.5)
- moved C4 6.63 mm to (207.5, 34.0)
- moved C3 6.54 mm to (201.5, 25.5)
- moved IC1 6.39 mm to (204.7, 29.0), turned to 90 degrees
- moved R2 4.12 mm to (210.0, 32.0), turned to 90 degrees
- moved C9 3.96 mm to (189.5, 17.4)
- moved C8 2.54 mm to (189.5, 13.9)
- moved U2 2.14 mm to (186.8, 14.6)
- moved C10 2.13 mm to (186.2, 17.2)
- moved D19 1.67 mm to (172.8, 24.8)
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Connections:
- D46 pad 1: unconnected-(D46-K1-Pad1) -> D-
- D46 pad 3: D- -> D+
- D46 pad 4: D+ -> unconnected-(D46-K3-Pad4)
- IC1 pad 10: unconnected-(IC1-PA4-Pad10) -> C8
- IC1 pad 11: unconnected-(IC1-PA5-Pad11) -> C7
- IC1 pad 12: unconnected-(IC1-PA6-Pad12) -> C6
- IC1 pad 13: unconnected-(IC1-PA7-Pad13) -> C5
- IC1 pad 14: unconnected-(IC1-PB0-Pad14) -> C4
- IC1 pad 15: unconnected-(IC1-PB1-Pad15) -> L2
- IC1 pad 16: unconnected-(IC1-PB2-Pad16) -> L1
- IC1 pad 18: L4 -> C3
- IC1 pad 19: L3 -> C2
- IC1 pad 2: L1 -> unconnected-(IC1-PC14-OSC32_IN-Pad2)
- IC1 pad 20: L2 -> C1
- IC1 pad 25: C10 -> unconnected-(IC1-PA15-Pad25)
- IC1 pad 26: C9 -> unconnected-(IC1-PB3-Pad26)
- IC1 pad 27: C8 -> unconnected-(IC1-PB4-Pad27)
- IC1 pad 28: C7 -> C11
- IC1 pad 29: C6 -> L4
- IC1 pad 3: C1 -> unconnected-(IC1-PC15-OSC32_OUT-Pad3)
- IC1 pad 30: C5 -> L3
- IC1 pad 32: C3 -> unconnected-(IC1-PB8-Pad32)
- IC1 pad 6: C4 -> unconnected-(IC1-PA0-Pad6)
- IC1 pad 7: C2 -> unconnected-(IC1-PA1-Pad7)
- IC1 pad 8: C11 -> C10
- IC1 pad 9: unconnected-(IC1-PA3-Pad9) -> C9
Routing:
- net 3V3N: track 72.1 -> 49.5 mm, vias 2 -> 5
- net +3.3V: track 15.9 -> 35.6 mm, vias 3 -> 5
- net C2: track 244.2 -> 225.6 mm, vias 4 -> 2
- net D-: track 31.7 -> 15.5 mm, vias 3 -> 2
- net SWCLK: track 40.9 -> 25.7 mm, vias 2 -> 1
- net C4: track 197.1 -> 185.3 mm, vias 3 -> 0
- net C7: track 135.0 -> 124.4 mm, vias 3 -> 0
- net C6: track 152.3 -> 145.3 mm, vias 3 -> 0
- net C9: track 91.7 -> 84.7 mm, vias 3 -> 0
- net C5: track 171.3 -> 164.7 mm, vias 3 -> 0
- net C8: track 111.3 -> 105.1 mm, vias 3 -> 0
- net L4: track 251.1 -> 257.3 mm
- net SWDIO: track 34.8 -> 29.0 mm, vias 4 -> 1
- net C10: track 68.8 -> 63.1 mm
- net C11: track 62.8 -> 68.4 mm
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- added copper zone on In2.Cu, net +3.3V
- added copper zone on In1.Cu, net GND
- removed copper zone on In1.Cu, net +3.3V
- removed copper zone on In2.Cu, net GND
Other:
- board text added: "A"
- board text added: "ALT"
- board text added: "B"
- board text added: "By (139 + 11) ^ 217"
- board text added: "C"
- board text added: "C1"
- board text added: "C10"
- board text added: "C11"
- board text added: "C2"
- board text added: "C3"
- board text added: "C4"
- board text added: "C5"
- board text added: "C6"
- board text added: "C7"
- board text added: "C8"
- board text added: "C9"
- board text added: "CTRL"
- board text added: "D"
- board text added: "DEL"
- board text added: "DOWN"
- board text added: "ENTER"
- board text added: "ESC"
- board text added: "F"
- board text added: "FN1"
- board text added: "FN2"
- board text added: "FN3"
- board text added: "FN4"
- board text added: "G"
- board text added: "H"
- board text added: "I"
- board text added: "J"
- board text added: "K"
- board text added: "L"
- board text added: "L1"
- board text added: "L2"
- board text added: "L3"
- board text added: "L4"
- board text added: "LEFT"
- board text added: "M"
- board text added: "N"
- board text added: "O"
- board text added: "P"
- board text added: "PA10 20"
- board text added: "PA2 8"
- board text added: "PA3 9"
- board text added: "PA4 10"
- board text added: "PA5 11"
- board text added: "PA6 12"
- board text added: "PA7 13"
- board text added: "PA8 18"
- board text added: "PA9 19"
- board text added: "PB0 14"
- board text added: "PB1 15"
- board text added: "PB2 16"
- board text added: "PB5 28"
- board text added: "PB6 29"
- board text added: "PB7 30"
- board text added: "Q"
- board text added: "R"
- board text added: "RIGHT"
- board text added: "S"
- board text added: "SHIFT"
- board text added: "SPACE"
- board text added: "SUPER"
- board text added: "SUPPR"
- board text added: "T"
- board text added: "TAB"
- board text added: "U"
- board text added: "UP"
- board text added: "V"
- board text added: "W"
- board text added: "X"
- board text added: "Y"
- board text added: "Z"

Commit message: readme
Parts:
- moved B17 52.4 mm to (131.6, 59.7)
- moved B18 52.4 mm to (131.6, 79.0)
- moved B19 52.4 mm to (131.6, 98.3)
- moved B20 52.4 mm to (131.6, 117.6)
- moved B21 52.4 mm to (150.9, 59.7)
- moved B22 52.4 mm to (150.9, 79.0)
- moved B23 52.4 mm to (150.9, 98.3)
- moved B24 52.4 mm to (150.9, 117.6)
- moved B25 52.4 mm to (170.2, 59.7)
- moved B26 52.4 mm to (170.2, 79.0)
- moved B27 52.4 mm to (170.2, 98.3)
- moved B28 52.4 mm to (170.2, 117.6)
- moved B29 52.4 mm to (189.5, 59.7)
- moved B30 52.4 mm to (189.5, 79.0)
- moved B31 52.4 mm to (189.5, 98.3)
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