File: elec/keyboard_steamdeck.kicad_pcb (KiCad board)
At the start: 4 copper layers, 213.4 x 77.8 mm, 112 parts, among them IC1 STM32L052K8U6TR, J2 STLINKV2 - DNI, J3 USB_C_Receptacle_USB2.0, U2 AP63203WU

Commit message: ready to order PCB
Parts:
- moved B12 45.0 mm to (122.7, 132.1)
- moved B9 45.0 mm to (103.4, 132.1)
- moved B15 45.0 mm to (142.0, 132.1)
- moved B19 45.0 mm to (161.3, 132.1)
- moved B23 45.0 mm to (180.6, 132.1)
- moved B27 45.0 mm to (199.9, 132.1)
- moved B31 45.0 mm to (219.2, 132.1)
- moved B35 45.0 mm to (238.5, 132.1)
- moved B39 45.0 mm to (257.8, 132.1)
- moved B43 45.0 mm to (277.1, 132.1)
- moved B6 45.0 mm to (84.1, 132.1)
- moved H1 45.0 mm to (110.5, 146.8)
- moved H4 45.0 mm to (245.6, 146.8)
- moved B11 45.0 mm to (122.7, 112.8)
- moved B3 45.0 mm to (103.4, 93.5)
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Routing:
- net +3.3V: track 35.6 -> 36.2 mm
- net GND: vias 725 -> 723
Other:
- board size 213.4 x 77.8 mm -> 213.4 x 77.5 mm
- board text added: "PA10 20 C11"
- board text added: "PA2 8 C10"
- board text added: "PA3 9 C9"
- board text added: "PA4 10 C8"
- board text added: "PA5 11 C7"
- board text added: "PA6 12 C6"
- board text added: "PA7 13 C5"
- board text added: "PA8 18 C3"
- board text added: "PA9 19 C2"
- board text added: "PB0 14 C4"
- board text added: "PB1 15 L2"
- board text added: "PB2 16 L1"
- board text added: "PB5 28 C11"
- board text added: "PB6 29 L4"
- board text added: "PB7 30 L3"
- board text removed: "C1"
- board text removed: "C10"
- board text removed: "C11"
- board text removed: "C2"
- board text removed: "C3"
- board text removed: "C4"
- board text removed: "C5"
- board text removed: "C6"
- board text removed: "C7"
- board text removed: "C8"
- board text removed: "C9"
- board text removed: "L1"
- board text removed: "L2"
- board text removed: "L3"
- board text removed: "L4"
- board text removed: "PA10 20"
- board text removed: "PA2 8"
- board text removed: "PA3 9"
- board text removed: "PA4 10"
- board text removed: "PA5 11"
- board text removed: "PA6 12"
- board text removed: "PA7 13"
- board text removed: "PA8 18"
- board text removed: "PA9 19"
- board text removed: "PB0 14"
- board text removed: "PB1 15"
- board text removed: "PB2 16"
- board text removed: "PB5 28"
- board text removed: "PB6 29"
- board text removed: "PB7 30"
