File: elec/keyboard_steamdeck.kicad_pcb (KiCad board)
At the start: 4 copper layers, 213.4 x 77.5 mm, 112 parts, among them IC1 STM32L052K8U6TR, J2 STLINKV2 - DNI, J3 USB_C_Receptacle_USB2.0, U2 AP63203WU

Commit message: working_key_scan
Routing:
- net C3: track 205.3 -> 205.9 mm
- net GND: vias 723 -> 719
Other:
- board text added: "PA10 20 C1"
- board text removed: "PA10 20 C11"
